File: wiring/ecu-masters-adu-dash-wiring/ecu-masters-adu-dash-wiring.kicad_sch (KiCad schematic)
At the start: 0 parts

Commit message: Adding a bunch of updates.
Parts:
- added J?: ADU_to_Car_Sensors, symbol ecu_masters:ADU_to_Car_Sensors
- added J?: USB_A, symbol Connector:USB_A
- added J?: ADU_to_ECU_Connector, symbol ecu_masters:ADU_to_ECU_Connector
- added J?: ADU_Connector, symbol ecu_masters:ADU_Connector
- added J?: ADU_to_Car_Signals, symbol ecu_masters:ADU_to_Car_Signals
Connections:
- new net: J?.1 (Fuel_Sender_Signal), J?.17 (Analog_In_A1)
- new net: J?.2 (Fuel_Sender_Ground), J?.4 (Coolant_Temp_Ground), J?.9 (Sensor_Ground)
- new net: J?.28 (Analog_In_A2), J?.3 (Coolant_Temp_Signal)
- new net: J?.1 (VBUS), J?.2 (USB.VBUS)
- new net: J?.13 (USB.DM), J?.2 (D-)
- new net: J?.14 (USB.DP), J?.3 (D+)
- new net: J?.1 (USB.GND), J?.4 (GND), J?.5 (Shield)
- new net: J?.1 (Power_Ground), J?.22 (Power_Ground)
- new net: J?.2 (Ground), J?.23 (Ground)
- new net: J?.3 (CAN1.H), J?.3 (CAN1.H)
- new net: J?.4 (CAN1.L), J?.4 (CAN1.L)
- new net: J?.11 (Switched_12V), J?.5 (Switched_12V)
- new net: J?.12 (Battery_12V), J?.6 (Battery_12V)
- new net: J?.18 (Digital_In_D8), J?.8 (Door_Ajar)
- new net: J?.19 (Digital_In_D6), J?.9 (Hand_Brake)
- new net: J?.20 (Digital_In_D4), J?.4 (High_Beams)
- new net: J?.2 (Right_Turn), J?.21 (Digital_In_D2)
- new net: J?.24 (Analog_In_A8), J?.6 (Low_Oil_Pressure)
- new net: J?.25 (Analog_In_A7), J?.7 (Low_PS_Pressure)
- new net: J?.10 (Cruise_Active), J?.30 (Digital_In_D7)
- new net: J?.31 (Digital_In_D5), J?.5 (No_Charging)
- new net: J?.3 (Headlights), J?.32 (Digital_In_D3)
- new net: J?.1 (Left_Turn), J?.33 (Digital_In_D1)
Other:
- note added: "BLK"
- note added: "Coolant Line Temp Sensor ~? ohms @ ~100 C (~212 F) ~? ohms @ ~20 C (~68 F)"
- note added: "Fuel Sender ~4 ohms full ~107 ohms empty"
- note added: "Is a low value external pullup needed?"
- note added: "ORA"
- note added: "PUR"
- note added: "RED"
- note added: "Twisted Pair"
- note added: "YLW"
